Commit message: update some topics name.

File: Car_Sim2Real/install/robot_description/share/robot_description/urdf/装配体2.SLDASM.urdf (robot description, URDF)
Before this commit: robot robot_description, 3 links, 2 joints
Joints:
- joint Laser_Joint: origin xyz=0 0 0.122512 rpy=0 0 3.1415926 -> xyz=0 0 0.122512 rpy=0 0 0
